Commit message: unicode error fixed

File: mybot_description/urdf/macros.xacro (robot description, xacro)
@@ -1,4 +1,21 @@
 <?xml version="1.0"?>
+ <robot>
+<macro name="cylinder_inertia" params="m r h">
+  <inertia  ixx="${m*(3*r*r+h*h)/12}" ixy = "0" ixz = "0"
+    iyy="${m*(3*r*r+h*h)/12}" iyz = "0"
+    izz="${m*r*r/2}"
+  />
+</macro>
 <macro name="box_inertia" params="m x y z">
-<inertia ixx="${m(y*y+z*z)/12}" ixy="0" ixz="0" iyy="${m(x*x+z*z)/12}" iyz="0" izz="${m*(y*y+x*x)/12}" />
+  <inertia  ixx="${m*(y*y+z*z)/12}" ixy = "0" ixz = "0"
+    iyy="${m*(x*x+z*z)/12}" iyz = "0"
+    izz="${m*(x*x+z*z)/12}"
+  />
 </macro>
+<macro name="sphere_inertia" params="m r">
+  <inertia  ixx="${2*m*r*r/5}" ixy = "0" ixz = "0"
+    iyy="${2*m*r*r/5}" iyz = "0"
+    izz="${2*m*r*r/5}"
+  />
+</macro>
+ </robot>

File: mybot_description/urdf/materials.xacro (robot description, xacro)
@@ -1,4 +1,27 @@
 <?xml version="1.0"?>
+<robot>
+<material name="black">
+  <color rgba="0.0 0.0 0.0 1.0"/>
+</material>
+<material name="blue">
+  <color rgba="0.0 0.0 0.8 1.0"/>
+</material>
+<material name="green">
+  <color rgba="0.0 0.8 0.0 1.0"/>
+</material>
+<material name="grey">
+  <color rgba="0.2 0.2 0.2 1.0"/>
+</material>
 <material name="orange">
- <color rgba="0.0 0.0 0.0 1.0"/>
+  <color rgba="${255/255} ${108/255} ${10/255} 1.0"/>
 </material>
+<material name="brown">
+  <color rgba="${222/255} ${207/255} ${195/255} 1.0"/>
+</material>
+<material name="red">
+  <color rgba="0.8 0.0 0.0 1.0"/>
+</material>
+<material name="white">
+  <color rgba="1.0 1.0 1.0 1.0"/>
+</material>
+</robot>

File: mybot_description/urdf/mybot.urdf.xacro (robot description, xacro)
@@ -15,19 +15,17 @@
 <xacro:property name="cameraMass" value="0.1"/>
 <xacro:include filename="$(find mybot_description)/urdf/mybot.gazebo" /> <!--all the gazebo-specific aspects of our robot-->
-<!--<xacro:include filename="$(find mybot_description)/urdf/materials.xacro" />definition of the materials used (mostly colors)-->
-<!-- <xacro:include filename="$(find mybot_description)/urdf/macros.xacro" /> definitions of some macros for easier description of the robot -->
-<material name="orange">
- <color rgba="0.0 0.0 0.0 1.0"/>
-</material>
-<macro name="box_inertia" params="m x y z">
-	<mass value="${m}"/>
-	<inertia ixx="${m*(z*z+y*y)*0.083}" ixy="0" ixz="0" iyy="${m*(x*x+z*z)*0.083}" iyz="0" izz="{m*(x*x+y*y)*0.083}"  />
-</macro>
+<xacro:include filename="$(find mybot_description)/urdf/materials.xacro" />
+<xacro:include filename="$(find mybot_description)/urdf/macros.xacro" />
+<link name="footprint"/>
+<joint name="base_joint" type="fixed">
+	<parent link="footprint"/>
+	<child link="chassis"/>
+</joint>
 <link name="chassis">
- <collision>
-	<origin xyz="0 0 ${wheelRadius}" rpy="0 0 0" />
-	<geometry>
-		<box size="${chassisLength} ${chassisWidth} ${chassisHeight}"/>
-	</geometry>
+  <collision>
+    <origin xyz="0 0 ${wheelRadius}" rpy="0 0 0"/>
+    <geometry>
+      <box size="${chassisLength} ${chassisWidth} ${chassisHeight}"/>
+    </geometry>
  </collision>
  <visual>
@@ -38,14 +36,9 @@
 	<material name="orange"/>
  </visual>
- <inertial>
+<inertial>
 	<origin xyz="0 0 ${wheelRadius}" rpy="0 0 0" />
 	<mass value="${chassisMass}"/>
-	<box_inertia m="${chassisMass}" x="{chassisLength}" y="${chassisWidth}" z="${chassisHeight}"/>
- </inertial>
+	<box_inertia m="${chassisMass}" x="${chassisLength}" y="${chassisWidth}" z="${chassisHeight}"/>
+</inertial>
 </link>
-<link name="footprint"/>
-<joint name="base_joint" type="fixed">
-	<parent link="footprint"/>
-	<child link="chassis"/>
-</joint>
 </robot>

File: mybot_description/urdf/mybot.xacro (robot description, xacro)
@@ -21,5 +21,5 @@
 </material>
 <macro name="box_inertia" params="m x y z">
-  <inertia  ixx="${m*(y*y+z*z)/12}" ixy="0" ixz="0" iyy="${m*(x*x+z*z)/12}" iyz="0" izz="${m*(x*x+z*z)/12}"/>
+  <inertia  ixx="0.001" ixy="0" ixz="0" iyy="0.001" iyz="0" izz="0.001"/>
 </macro>
 <link name="chassis">
